File: MiniArcade_MainBoard/MiniArcade_MainBoard.kicad_sch (KiCad schematic)
At the start: 30 parts, among them J1 62701021721, J2 Conn_01x05_Pin, J3 Conn_01x06_Pin, J4 F3311A7H121026E200, SW1 EVPAA, U1 ATSAMD21J18A-A, U2 LM321

Commit message: title and Author added
Other:
- company: (none) -> Felix Neumann
- title: (none) -> MiniArcadeMainboard
Changed lines of the file:
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@@
 	(generator_version "9.0")
 	(paper "A4")
+	(title_block
+		(title "MiniArcadeMainboard")
+		(date "2025-10-29")
+		(rev "A")
+		(company "Felix Neumann")
+	)
 	(rectangle
 		(start 101.6 13.97)
