File: MiniArcade_MainBoard/MiniArcade_MainBoard.kicad_sch (KiCad schematic)
At the start: 30 parts, among them J1 62701021721, J2 Conn_01x05_Pin, J3 Conn_01x06_Pin, J4 F3311A7H121026E200, SW1 EVPAA, U1 ATSAMD21J18A-A, U2 LM321

Commit message: stand 03 11
Connections:
- net +3.3V: no longer J1.1
- net 3.3V: no longer C10.1, C11.1, C6.1, C7.1, C9.1, FB1.1, U1.21 (VDDIO), U1.34 (VDDIO), U1.48 (VDDIO), U1.56 (VDDIN)
- net 3V3: now also C10.1, C11.1, C6.1, C7.1, C9.1, FB1.1, J1.1, U1.21 (VDDIO), U1.34 (VDDIO), U1.48 (VDDIO), U1.56 (VDDIN)
- net BUZZER: now also U1.59 (PB30); no longer U1.5 (PB04)
- net GND: now also J4.10, J4.11, J4.12, J4.13, J4.14, J4.15, J4.16, J4.19
- net RESET: no longer J4.18, U1.10 (PB07)
- net SCWCLK renamed SWCLK
- net VDD renamed LCD_VDD
- net VDDI renamed LCD_VDDI
- new net LCD_RESET: J4.18, U1.10 (PB07)
- no-connect marks 55 -> 42
Other:
- note added: "Buzzer VIN: -1,5V to +1,5V SAMD21 PB30: Squarewave 0V to 3,3V Solution: Virtual Ground @ 1,65V"
- note added: "Pins 1 bis 4 für Touchpannel, garnicht vorhanden bei der LCD Variante. Auf GND oder nicht verbunden?"
- note removed: "Buzzer VIN: -1,5V to +1,5V SAMD21 PB04: Squarewave 0V to 3,3V Solution: Virtual Ground @ 1,65V"
- note removed: "Stecker SMD Buchse THT"
- note removed: "unbenutze Pins auf GND?"
- moved on the sheet: J4

Commit message: stand 04 11 2025
Connections:
- net BLA: now also U1.12 (PB09); no longer U1.63 (PB02)
- net BUZZER: now also U1.13 (PA04); no longer U1.59 (PB30)
- net CS: now also U1.11 (PB08); no longer U1.6 (PB05)
- net DC: now also U1.6 (PB05); no longer U1.64 (PB03)
- net DP_DOWN: now also U1.29 (PA12)
- net DP_LEFT: now also U1.28 (PB15)
- net DP_RIGHT: now also U1.30 (PA13)
- net DP_UP: now also U1.31 (PA14)
- net JS_DOWN: now also U1.39 (PB16)
- net JS_LEFT: now also U1.40 (PB17)
- net JS_RIGHT: now also U1.37 (PA18)
- net JS_SWITCH: now also U1.38 (PA19)
- net JS_UP: now also U1.41 (PA20)
- net LCD_RESET: now also U1.4 (PA03); no longer U1.10 (PB07)
- net LCD_VDD: now also U1.1 (PA00); no longer U1.61 (PB00)
- net LCD_VDDI: now also U1.2 (PA01); no longer U1.62 (PB01)
- net SPI4W: now also U1.3 (PA02); no longer U1.9 (PB06)
- net USER_LED: now also U1.32 (PA15)
- no-connect marks 42 -> 38

Commit message: 05 11 2025
Other:
- note added: "<-LCD_VDD"
- note added: "<-LCD_VDDI"
- note added: "LCD VDD & VDDI liegen in MPLAB noch auf PB00 & PB01"
Changed lines of the file:
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@@
+		)
+	)
+	(text "LCD VDD & VDDI \nliegen in MPLAB noch \nauf PB00 & PB01"
+		(exclude_from_sim no)
+		(at 256.032 56.388 0)
+		(effects
+			(font
+				(size 1.27 1.27)
+				(color 255 25 41 1)
+			)
+			(justify left)
 		)
 	)
@@
 			)
 			(justify left bottom)
+		)
+	)
+	(text "<-LCD_VDD"
+		(exclude_from_sim no)
+		(at 258.572 49.53 0)
+		(effects
+			(font
+				(size 1.27 1.27)
+				(color 255 25 41 1)
+			)
 		)
 	)
@@
 		)
 	)
+	(text "<-LCD_VDDI\n\n"
+		(exclude_from_sim no)
+		(at 258.826 53.34 0)
+		(effects
+			(font
+				(size 1.27 1.27)
+				(color 255 25 41 1)
+			)
+		)
+	)

Commit message: 10 11 2025
Connections:
- net LCD_RESET: now also U1.5 (PB04); no longer U1.4 (PA03)
Changed lines of the file:
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@@
 	(text "LCD VDD & VDDI \nliegen in MPLAB noch \nauf PB00 & PB01"
 		(exclude_from_sim no)
-		(at 256.032 56.388 0)
+		(at 256.032 55.88 0)
 		(effects
 			(font
@@
 	)
 	(no_connect
-		(at 251.46 59.69)
-	)
-	(no_connect
 		(at 251.46 128.27)
 	)
@@
 	)
 	(no_connect
+		(at 215.9 57.15)
+	)
+	(no_connect
 		(at 83.82 45.72)
 	)
@@
 	(wire
 		(pts
-			(xy 208.28 57.15) (xy 215.9 57.15)
-		)
-		(stroke
-			(width 0)
-			(type default)
-		)
-	)
-	(wire
-		(pts
 			(xy 111.76 71.12) (xy 111.76 73.66)
 		)
@@
 	(wire
 		(pts
+			(xy 251.46 59.69) (xy 256.54 59.69)
+		)
+		(stroke
+			(width 0)
+			(type default)
+		)
+	)
+	(wire
+		(pts
 			(xy 143.51 43.18) (xy 160.02 43.18)
 		)
@@
 		)
 	)
-	(global_label "LCD_RESET"
-		(shape input)
-		(at 208.28 57.15 180)
-		(fields_autoplaced yes)
-		(effects
-			(font
-				(size 1.27 1.27)
-			)
-			(justify right)
-		)
-		(property "Intersheetrefs" "${INTERSHEET_REFS}"
-			(at 195.014 57.15 0)
-			(effects
-				(font
-					(size 1.27 1.27)
-				)
-				(justify right)
-				(hide yes)
-			)
-		)
-	)
 	(global_label "GND"
 		(shape input)
@@
 		)
 	)
+	(global_label "LCD_RESET"
+		(shape input)
+		(at 256.54 59.69 0)
+		(fields_autoplaced yes)
+		(effects
+			(font
+				(size 1.27 1.27)
+			)
+			(justify left)
+		)
+		(property "Intersheetrefs" "${INTERSHEET_REFS}"
+			(at 269.806 59.69 0)
+			(effects
+				(font
+					(size 1.27 1.27)
+				)
+				(justify left)
+				(hide yes)
+			)
+		)
+	)
 	(global_label "JS_SWITCH"
 		(shape input)
@@
 		(dnp no)
 		(property "Reference" "C4"
-			(at 151.13 121.92 0)
+			(at 161.544 121.92 0)
 			(effects
 				(font
@@
 		)
 		(property "Value" "100p"
-			(at 152.4 124.46 0)
+			(at 162.814 124.46 0)
 			(effects
 				(font

Commit message: 11 11 2025
Parts:
- added U3: ~, MainBoard:ERTFT144, symbol MainBoard:ERTFT144
- J2: footprint Connector_PinHeader_1.00mm:PinHeader_1x05_P1.00mm_Horizontal -> Connector_PinHeader_2.54mm:PinHeader_1x05_P2.54mm_Vertical
- J3: footprint Connector_PinHeader_1.00mm:PinHeader_1x06_P1.00mm_Horizontal -> Connector_PinHeader_2.54mm:PinHeader_1x06_P2.54mm_Vertical
Connections:
- net +3.3V is gone; now on net 3V3: R7.2
- net 3.3V is gone; now on net 3V3: C4.1, R4.1
- no-connect marks 38 -> 64
Other:
- note added: "FPC-Connector: 26 Pin 0.5 mm Pitch Dual Connection LCD -> ERTFT144-1"
- note added: "LCD ER-TFT1.44-1"
- note removed: "FPC-Connector: 26 Pin 0.5 mm Pitch Bottom Connection LCD -> ERTFT144-1"
Changed lines of the file:
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@@
 	)
 	(rectangle
+		(start 12.7 13.97)
+		(end 55.88 113.03)
+		(stroke
+			(width 0)
+			(type dash)
+		)
+		(fill
+			(type none)
+		)
+	)
+	(rectangle
 		(start 101.6 13.97)
 		(end 175.26 82.55)
@@
 		)
 	)
+	(text "LCD ER-TFT1.44-1\n"
+		(exclude_from_sim no)
+		(at 23.114 16.002 0)
+		(effects
+			(font
+				(size 1.27 1.27)
+			)
+		)
+	)
 	(text "LED Pin noch\nauf SAMD21 legen\n"
 		(exclude_from_sim no)
@@
 		)
 	)
-	(text "FPC-Connector:\n	26 Pin 0.5 mm Pitch\n	Bottom Connection\n	LCD -> ERTFT144-1"
+	(text "FPC-Connector:\n26 Pin 0.5 mm Pitch\nDual Connection\nLCD -> ERTFT144-1"
 		(exclude_from_sim no)
-		(at 66.802 19.812 0)
+		(at 57.912 19.05 0)
 		(effects
 			(font
 				(size 1.27 1.27)
 			)
+			(justify left)
 		)
 	)
@@
 	)
 	(no_connect
+		(at 46.99 59.69)
+	)
+	(no_connect
 		(at 251.46 82.55)
 	)
@@
 	)
 	(no_connect
+		(at 46.99 41.91)
+	)
+	(no_connect
 		(at 215.9 62.23)
 	)
@@
 	)
 	(no_connect
+		(at 46.99 97.79)
+	)
+	(no_connect
+		(at 46.99 64.77)
+	)
+	(no_connect
 		(at 83.82 43.18)
 	)
 	(no_connect
+		(at 46.99 46.99)
+	)
+	(no_connect
+		(at 46.99 54.61)
+	)
+	(no_connect
 		(at 215.9 69.85)
 	)
@@
 	)
 	(no_connect
+		(at 46.99 69.85)
+	)
+	(no_connect
 		(at 157.48 99.06)
 	)
@@
 	)
 	(no_connect
+		(at 46.99 49.53)
+	)
+	(no_connect
 		(at 251.46 128.27)
 	)
 	(no_connect
+		(at 46.99 52.07)
+	)
+	(no_connect
 		(at 251.46 57.15)
 	)
@@
 	)
 	(no_connect
+		(at 46.99 95.25)
+	)
+	(no_connect
 		(at 251.46 49.53)
 	)
@@
 	)
 	(no_connect
+		(at 46.99 74.93)
+	)
+	(no_connect
 		(at 83.82 96.52)
 	)
 	(no_connect
+		(at 46.99 92.71)
+	)
+	(no_connect
 		(at 215.9 105.41)
 	)
@@
 	)
 	(no_connect
+		(at 46.99 72.39)
+	)
+	(no_connect
 		(at 251.46 67.31)
 	)
@@
 	)
 	(no_connect
+		(at 46.99 57.15)
+	)
+	(no_connect
 		(at 215.9 110.49)
 	)
 	(no_connect
+		(at 46.99 77.47)
+	)
+	(no_connect
 		(at 251.46 64.77)
 	)
 	(no_connect
+		(at 46.99 100.33)
+	)
+	(no_connect
 		(at 58.42 40.64)
 	)
 	(no_connect
+		(at 46.99 85.09)
+	)
+	(no_connect
+		(at 46.99 80.01)
+	)
+	(no_connect
 		(at 215.9 107.95)
 	)
 	(no_connect
+		(at 46.99 87.63)
+	)
+	(no_connect
 		(at 251.46 54.61)
 	)
@@
 	)
 	(no_connect
+		(at 46.99 44.45)
+	)
+	(no_connect
 		(at 215.9 120.65)
 	)
 	(no_connect
+		(at 46.99 62.23)
+	)
+	(no_connect
+		(at 46.99 102.87)
+	)
+	(no_connect
 		(at 215.9 92.71)
 	)
@@
 	)
 	(no_connect
+		(at 46.99 67.31)
+	)
+	(no_connect
+		(at 46.99 82.55)
+	)
+	(no_connect
+		(at 46.99 105.41)
+	)
+	(no_connect
 		(at 83.82 48.26)
 	)
+	(no_connect
+		(at 46.99 90.17)
+	)
 	(wire
 		(pts
@@
 		)
 	)
-	(global_label "+3.3V"
+	(global_label "3V3"
 		(shape input)
 		(at 200.66 116.84 180)
@@
 		)
 		(property "Intersheetrefs" "${INTERSHEET_REFS}"
-			(at 191.99 116.84 0)
+			(at 194.1672 116.84 0)
 			(effects
 				(font
@@
 		)
 	)
-	(global_label "3.3V"
+	(global_label "3V3"
 		(shape input)
 		(at 148.59 116.84 0)
@@
 		)
 		(property "Intersheetrefs" "${INTERSHEET_REFS}"
-			(at 155.6876 116.84 0)
+			(at 155.0828 116.84 0)
 			(effects
 				(font
@@
 			)
 		)
-		(property "Footprint" "Connector_PinHeader_1.00mm:PinHeader_1x05_P1.00mm_Horizontal"
+		(property "Footprint" "Connector_PinHeader_2.54mm:PinHeader_1x05_P2.54mm_Vertical"
 			(at 58.42 132.08 0)
 			(effects
@@
 	)
 	(symbol
+		(lib_id "MainBoard:ERTFT144")
+		(at 34.29 39.37 0)
+		(unit 1)
+		(exclude_from_sim no)
+		(in_bom yes)
+		(on_board yes)
+		(dnp no)
+		(property "Reference" "U3"
+			(at 33.02 19.05 0)
+			(effects
+				(font
+					(size 1.27 1.27)
+				)
+			)
+		)
+		(property "Value" "~"
+			(at 33.02 17.78 0)
+			(effects
+				(font
+					(size 1.27 1.27)
+				)
+				(hide yes)
+			)
+		)
+		(property "Footprint" "MainBoard:ERTFT144"
+			(at 34.29 39.37 0)
+			(effects
+				(font
+					(size 1.27 1.27)
+				)
+				(hide yes)
+			)
+		)
+		(property "Datasheet" ""
+			(at 34.29 39.37 0)
+			(effects
+				(font
+					(size 1.27 1.27)
+				)
+				(hide yes)
+			)
+		)
+		(property "Description" ""
+			(at 34.29 39.37 0)
+			(effects
+				(font
+					(size 1.27 1.27)
+				)
+				(hide yes)
+			)
+		)
+		(pin "9"
+		)
+		(pin "11"
+		)
+		(pin "17"
+		)
+		(pin "26"
+		)
+		(pin "7"
+		)
+		(pin "14"
+		)
+		(pin "16"
+		)
+		(pin "1"
+		)
+		(pin "6"
+		)
+		(pin "2"
+		)
+		(pin "8"
+		)
+		(pin "15"
+		)
+		(pin "19"
+		)
+		(pin "3"
+		)
+		(pin "10"
+		)
+		(pin "18"
+		)
+		(pin "22"
+		)
+		(pin "4"
+		)
+		(pin "5"
+		)
+		(pin "13"
+		)
+		(pin "21"
+		)
+		(pin "23"
+		)
+		(pin "24"
+		)
+		(pin "25"
+		)
+		(pin "12"
+		)
+		(pin "20"
+		)
+		(instances
+			(project ""
+				(path "/05ad7677-8bf5-470f-850e-ef78977ca036"
+					(reference "U3")
+					(unit 1)
+				)
+			)
+		)
+	)
+	(symbol
 		(lib_id "Device:C")
 		(at 154.94 124.46 0)
@@
 			)
 		)
-		(property "Footprint" "Connector_PinHeader_1.00mm:PinHeader_1x06_P1.00mm_Horizontal"
+		(property "Footprint" "Connector_PinHeader_2.54mm:PinHeader_1x06_P2.54mm_Vertical"
 			(at 80.01 132.08 0)
 			(effects

Commit message: 11 11 2025
Connections:
- no-connect marks 64 -> 66
Changed lines of the file:
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@@
+	)
+	(no_connect
+		(at 251.46 107.95)
 	)
 	(no_connect
@@
 	)
 	(no_connect
+		(at 251.46 105.41)
+	)
+	(no_connect

Commit message: 17 11 2025
Connections:
- net DP_DOWN: now also J2.4 (Pin_4), U1.38 (PA19); no longer J3.5 (Pin_5), U1.29 (PA12)
- net DP_LEFT: now also J2.5 (Pin_5), U1.37 (PA18); no longer J3.6 (Pin_6), U1.28 (PB15)
- net DP_RIGHT: now also J2.3 (Pin_3), U1.39 (PB16); no longer J3.4 (Pin_4), U1.30 (PA13)
- net DP_UP: now also J2.2 (Pin_2), U1.40 (PB17); no longer J3.3 (Pin_3), U1.31 (PA14)
- net GND: now also J2.1 (Pin_1); no longer J3.2 (Pin_2)
- net JS_DOWN: now also J3.4 (Pin_4), U1.29 (PA12); no longer J2.3 (Pin_3), U1.39 (PB16)
- net JS_LEFT: now also J3.3 (Pin_3), U1.30 (PA13); no longer J2.2 (Pin_2), U1.40 (PB17)
- net JS_RIGHT: now also J3.6 (Pin_6), U1.27 (PB14); no longer J2.5 (Pin_5), U1.37 (PA18)
- net JS_SWITCH: now also J3.5 (Pin_5), U1.28 (PB15); no longer J2.4 (Pin_4), U1.38 (PA19)
- net JS_UP: now also J3.2 (Pin_2), U1.31 (PA14); no longer J2.1 (Pin_1), U1.41 (PA20)

Commit message: 26 11 2025
Other:
- note removed: "Pins 1 bis 4 für Touchpannel, garnicht vorhanden bei der LCD Variante. Auf GND oder nicht verbunden?"
Changed lines of the file:
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@@
-		)
-	)
-	(text "Pins 1 bis 4 \nfür Touchpannel, garnicht vorhanden \nbei der LCD Variante.\nAuf GND oder nicht verbunden?\n"
-		(exclude_from_sim no)
-		(at 79.502 28.702 0)
-		(effects
-			(font
-				(size 1.27 1.27)
-				(color 255 21 54 1)
-			)
 		)
 	)
