File: MiniArcade_MainBoard/MiniArcade_MainBoard.kicad_sch (KiCad schematic)
At the start: 31 parts, among them J1 62701021721, J2 Conn_01x05_Pin, J3 Conn_01x06_Pin, J4 F3311A7H121026E200, SW1 EVPAA, U1 ATSAMD21J18A-A, U2 LM321

Commit message: 06 02 2026
Parts:
- R2: value R -> 330
Other:
- note removed: "LED Pin noch auf SAMD21 legen"
Changed lines of the file:
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@@
 		)
 	)
-	(text "LED Pin noch\nauf SAMD21 legen\n"
-		(exclude_from_sim no)
-		(at 73.406 167.386 0)
-		(effects
-			(font
-				(size 1.27 1.27)
-				(color 255 38 35 1)
-			)
-		)
-	)
 	(text "Reset Button:\n\n\n"
 		(exclude_from_sim no)
@@
 			)
 		)
-		(property "Value" "R"
+		(property "Value" "330"
 			(at 91.44 170.1799 0)
 			(effects
