File: MiniArcade_MainBoard/MiniArcade_MainBoard.kicad_pcb (KiCad board)
At the start: 2 copper layers, 30 parts, among them J1 62701021721, J2 Conn_01x05_Pin, J3 Conn_01x06_Pin, J4 F3311A7H121026E200, SW1 EVPAA, U1 ATSAMD21J18A-A, U2 LM321

Commit message: stand 03 11
Parts:
- moved R6 276.2 mm to (207.8, 146.0)
- moved C2 274.3 mm to (207.8, 148.0)
- moved FB1 255.6 mm to (188.9, 118.8), turned to 180 degrees
- moved C1 252.4 mm to (181.2, 155.6), turned to 180 degrees
- moved R3 251.9 mm to (176.0, 157.6)
- moved R5 250.6 mm to (176.0, 159.6), turned to 180 degrees
- moved C3 248.8 mm to (188.9, 121.0)
- moved LS1 248.2 mm to (195.5, 152.0), turned to 180 degrees
- moved U2 247.2 mm to (181.2, 158.6)
- moved R2 246.1 mm to (182.5, 108.2), turned to 90 degrees
- moved C6 244.0 mm to (185.0, 124.5)
- moved C9 243.2 mm to (188.9, 116.5), turned to 180 degrees
- moved C5 238.2 mm to (177.2, 130.8), turned to 180 degrees
- moved J4 238.0 mm to (176.5, 140.0)
- moved C11 232.6 mm to (179.5, 113.8), turned to 90 degrees
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Connections:
- net SCWCLK renamed SWCLK
- net VDD renamed LCD_VDD
- net VDDI renamed LCD_VDDI
- C10 pad 1: 3.3V -> 3V3
- C11 pad 1: 3.3V -> 3V3
- C6 pad 1: 3.3V -> 3V3
- C7 pad 1: 3.3V -> 3V3
- C9 pad 1: 3.3V -> 3V3
- FB1 pad 1: 3.3V -> 3V3
- J1 pad 1: +3.3V -> 3V3
- J4 pad 10: unconnected-(J4-Pad10) -> GND
- J4 pad 11: unconnected-(J4-Pad11) -> GND
- J4 pad 12: unconnected-(J4-Pad12) -> GND
- J4 pad 13: unconnected-(J4-Pad13) -> GND
- J4 pad 14: unconnected-(J4-Pad14) -> GND
- J4 pad 15: unconnected-(J4-Pad15) -> GND
- J4 pad 16: unconnected-(J4-Pad16) -> GND
- J4 pad 18: RESET -> LCD_RESET
- J4 pad 19: unconnected-(J4-Pad19) -> GND
- U1 pad 10: RESET -> LCD_RESET
- U1 pad 21: 3.3V -> 3V3
- U1 pad 34: 3.3V -> 3V3
- U1 pad 48: 3.3V -> 3V3
- U1 pad 5: BUZZER -> unconnected-(U1-PB04-Pad5)
- U1 pad 56: 3.3V -> 3V3
- U1 pad 59: unconnected-(U1-PB30-Pad59) -> BUZZER
Routing:
- net SWCLK: track 0.00 -> 25.5 mm
- net RESET: track 0.00 -> 20.5 mm
- net SWDIO: track 0.00 -> 12.6 mm
- net MOSI: track 0.00 -> 10.7 mm
- net SCLK: track 0.00 -> 10.3 mm
- net Net-(C4-Pad2): track 0.00 -> 6.55 mm
- net 3V3: track 0.00 -> 6.27 mm
- net VDDCORE: track 0.00 -> 4.91 mm
- net VDDANA: track 0.00 -> 3.71 mm
- net GNDANA: track 0.00 -> 2.63 mm
- net 1V65: track 0.00 -> 2.50 mm
- net Net-(R1-Pad1): track 0.00 -> 2.18 mm
- net Net-(U2-+): track 0.00 -> 2.00 mm
Other:
- board outline added: 55.5 x 42 mm

Commit message: stand 04 11 2025
Parts:
- moved R6 27.7 mm to (185.8, 129.2), turned to 180 degrees
- moved C2 27.5 mm to (185.8, 131.5)
- moved J2 27.2 mm to (151.4, 112.2)
- moved R5 24.2 mm to (188.8, 139.0), turned to 90 degrees
- moved U2 22.0 mm to (191.8, 139.2), turned to 90 degrees
- moved C1 21.5 mm to (189.8, 135.8)
- moved R3 21.4 mm to (186.5, 139.0), turned to -90 degrees
- moved LS1 20.4 mm to (198.2, 131.8), turned to -90 degrees
- moved SW1 18.8 mm to (155.8, 129.8), turned to -90 degrees
- moved R1 15.3 mm to (155.8, 126.0), turned to 180 degrees
- moved R4 13.8 mm to (155.8, 123.8), turned to 180 degrees
- moved C4 12.9 mm to (155.8, 121.5), turned to 180 degrees
- moved R10 12.8 mm to (155.8, 119.0), turned to 0 degrees
- moved J3 12.4 mm to (204.1, 116.8)
- moved J1 12.1 mm to (161.8, 135.1), turned to 0 degrees
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Connections:
- U1 pad 1: unconnected-(U1-PA00-Pad1) -> LCD_VDD
- U1 pad 10: LCD_RESET -> unconnected-(U1-PB07-Pad10)
- U1 pad 11: unconnected-(U1-PB08-Pad11) -> CS
- U1 pad 12: unconnected-(U1-PB09-Pad12) -> BLA
- U1 pad 13: unconnected-(U1-PA04-Pad13) -> BUZZER
- U1 pad 2: unconnected-(U1-PA01-Pad2) -> LCD_VDDI
- U1 pad 28: unconnected-(U1-PB15-Pad28) -> DP_LEFT
- U1 pad 29: unconnected-(U1-PA12-Pad29) -> DP_DOWN
- U1 pad 3: unconnected-(U1-PA02-Pad3) -> SPI4W
- U1 pad 30: unconnected-(U1-PA13-Pad30) -> DP_RIGHT
- U1 pad 31: unconnected-(U1-PA14-Pad31) -> DP_UP
- U1 pad 32: unconnected-(U1-PA15-Pad32) -> USER_LED
- U1 pad 37: unconnected-(U1-PA18-Pad37) -> JS_RIGHT
- U1 pad 38: unconnected-(U1-PA19-Pad38) -> JS_SWITCH
- U1 pad 39: unconnected-(U1-PB16-Pad39) -> JS_DOWN
- U1 pad 4: unconnected-(U1-PA03-Pad4) -> LCD_RESET
- U1 pad 40: unconnected-(U1-PB17-Pad40) -> JS_LEFT
- U1 pad 41: unconnected-(U1-PA20-Pad41) -> JS_UP
- U1 pad 59: BUZZER -> unconnected-(U1-PB30-Pad59)
- U1 pad 6: CS -> DC
- U1 pad 61: LCD_VDD -> unconnected-(U1-PB00-Pad61)
- U1 pad 62: LCD_VDDI -> unconnected-(U1-PB01-Pad62)
- U1 pad 63: BLA -> unconnected-(U1-PB02-Pad63)
- U1 pad 64: DC -> unconnected-(U1-PB03-Pad64)
- U1 pad 9: SPI4W -> unconnected-(U1-PB06-Pad9)
Routing:
- net JS_RIGHT: track 0.00 -> 33.2 mm
- net VDDANA: track 3.71 -> 36.1 mm, vias 0 -> 2
- net JS_SWITCH: track 0.00 -> 31.9 mm
- net JS_DOWN: track 0.00 -> 31.0 mm
- net JS_LEFT: track 0.00 -> 29.9 mm
- net JS_UP: track 0.00 -> 28.8 mm, vias 0 -> 2
- net DP_UP: track 0.00 -> 22.5 mm
- net DP_LEFT: track 0.00 -> 22.5 mm
- net DP_RIGHT: track 0.00 -> 22.3 mm
- net DP_DOWN: track 0.00 -> 22.3 mm
- net RESET: track 20.5 -> 38.9 mm
- net BLA: track 0.00 -> 16.6 mm, vias 0 -> 2
- net LCD_RESET: track 0.00 -> 15.3 mm, vias 0 -> 2
- net DC: track 0.00 -> 15.1 mm, vias 0 -> 2
- net Net-(C2-Pad2): track 0.00 -> 13.8 mm
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
Commit message: 10 11 2025
Connections:
- U1 pad 4: LCD_RESET -> unconnected-(U1-PA03-Pad4)
- U1 pad 5: unconnected-(U1-PB04-Pad5) -> LCD_RESET
Changed lines of the file:
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@@
 	(net 74 "unconnected-(U1-PB02-Pad63)")
 	(net 75 "unconnected-(U1-PB07-Pad10)")
-	(net 76 "unconnected-(U1-PB04-Pad5)")
+	(net 76 "unconnected-(U1-PA03-Pad4)")
 	(net 77 "unconnected-(U1-PB03-Pad64)")
 	(footprint "Resistor_SMD:R_0805_2012Metric_Pad1.20x1.40mm_HandSolder"
@@
 			(layers "F.Cu" "F.Mask" "F.Paste")
 			(roundrect_rratio 0.25)
-			(net 30 "LCD_RESET")
+			(net 76 "unconnected-(U1-PA03-Pad4)")
 			(pinfunction "PA03")
-			(pintype "bidirectional")
+			(pintype "bidirectional+no_connect")
 		)
 		(pad "5" smd roundrect
@@
 			(layers "F.Cu" "F.Mask" "F.Paste")
 			(roundrect_rratio 0.25)
-			(net 76 "unconnected-(U1-PB04-Pad5)")
+			(net 30 "LCD_RESET")
 			(pinfunction "PB04")
-			(pintype "bidirectional+no_connect")
+			(pintype "bidirectional")
 		)
 		(pad "6" smd roundrect
@@
 	)
 	(segment
-		(start 174 128.4125)
-		(end 174 134.5)
+		(start 178.75 139.227)
+		(end 178.75 138.575)
 		(width 0.2)
 		(layer "F.Cu")
@@
 	)
 	(segment
-		(start 178.75 139.227)
-		(end 178.75 138.575)
+		(start 174.5 128.4125)
+		(end 174.5 135)
 		(width 0.2)
 		(layer "F.Cu")
@@
 	)
 	(segment
-		(start 174 134.5)
+		(start 174.5 135)
 		(end 175.25 135.75)
 		(width 0.2)

Commit message: 11 11 2025
Parts:
- added U3: ~, MainBoard:ERTFT144, B.Cu at (155.3, 95.2)
- J2: footprint Connector_PinHeader_1.00mm:PinHeader_1x05_P1.00mm_Horizontal -> Connector_PinHeader_2.54mm:PinHeader_1x05_P2.54mm_Vertical
- J3: footprint Connector_PinHeader_1.00mm:PinHeader_1x06_P1.00mm_Horizontal -> Connector_PinHeader_2.54mm:PinHeader_1x06_P2.54mm_Vertical
- moved FB1 62.6 mm to (141.1, 135.8)
- moved C3 62.5 mm to (137.2, 135.8)
- moved J2 40.2 mm to (111.2, 115.2)
- moved NT1 40.1 mm to (136.2, 134.8)
- moved C10 40.1 mm to (132.8, 116.2)
- moved C11 40.1 mm to (139.5, 116.2)
- moved C4 40.1 mm to (115.8, 124.0)
- moved C5 40.1 mm to (137.2, 133.8)
- moved C6 40.1 mm to (145.0, 127.0)
- moved C7 40.1 mm to (126.0, 123.5)
- moved C8 40.1 mm to (126.0, 121.5)
- moved LED1 40.1 mm to (148.8, 115.8)
- moved R1 40.1 mm to (115.8, 128.5)
- moved R10 40.1 mm to (115.8, 121.5)
- moved R2 40.1 mm to (148.8, 118.2)
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Connections:
- C4 pad 1: 3.3V -> 3V3
- R4 pad 1: 3.3V -> 3V3
- R7 pad 2: +3.3V -> 3V3
Routing:
- net 3V3: track 19.0 -> 172.4 mm, vias 0 -> 8
- net GND: track 0.00 -> 29.2 mm, vias 0 -> 31
- net VDDANA: track 36.1 -> 7.82 mm, vias 2 -> 0
- net DP_UP: track 22.5 -> 31.8 mm
- net DP_RIGHT: track 22.3 -> 30.9 mm
- net DP_DOWN: track 22.3 -> 30.1 mm
- net DP_LEFT: track 22.5 -> 29.2 mm
- net JS_RIGHT: track 33.2 -> 39.6 mm
- net JS_SWITCH: track 31.9 -> 36.9 mm
- net CS: track 11.7 -> 16.2 mm
- net Net-(R1-Pad1): track 2.18 -> 5.54 mm
- net JS_DOWN: track 31.0 -> 34.1 mm
- net Net-(C2-Pad2): track 13.8 -> 16.6 mm
- net JS_UP: track 28.8 -> 30.9 mm, vias 2 -> 0
- net BUZZER: track 7.91 -> 9.81 mm
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- added copper zone on B.Cu, net GND
- added copper zone on F.Cu, net GND
Other:
- board size 55.5 x 42 mm -> 60 x 55 mm
- board text added: "Board: Mini Arcade Mainboard V1.0 Author: Felix Neumann Date: 11/11/2025"

Commit message: 11 11 2025
Parts:
- moved C9 18.3 mm to (145.5, 108.8), turned to 90 degrees
- moved C6 8.61 mm to (148.8, 119.2)
- moved U1 8.61 mm to (140.0, 117.5)
- moved C11 8.39 mm to (143.2, 108.8)
- moved FB1 8.32 mm to (143.0, 127.8), turned to 90 degrees
- moved C10 8.28 mm to (136.2, 108.8)
- moved C5 7.91 mm to (139.8, 126.2)
- moved C3 7.76 mm to (139.8, 128.5)
- moved NT1 7.69 mm to (138.8, 127.5)
- moved C7 7.40 mm to (130.0, 117.2)
- moved C8 7.40 mm to (130.0, 115.2)
- moved R7 7.40 mm to (130.0, 119.2)
- moved LS1 6.99 mm to (160.5, 128.2), turned to 0 degrees
- moved C2 6.46 mm to (150.2, 127.2), turned to -90 degrees
- moved C1 6.24 mm to (160.0, 137.5)
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Routing:
- net JS_LEFT: track 31.3 -> 41.9 mm
- net SWCLK: track 24.5 -> 34.9 mm
- net JS_DOWN: track 34.1 -> 43.5 mm
- net JS_SWITCH: track 36.9 -> 45.8 mm
- net JS_RIGHT: track 39.6 -> 48.2 mm
- net SWDIO: track 17.5 -> 26.1 mm
- net MOSI: track 11.1 -> 19.4 mm
- net JS_UP: track 30.9 -> 38.6 mm
- net DP_UP: track 31.8 -> 24.8 mm
- net DP_RIGHT: track 30.9 -> 24.0 mm
- net DP_DOWN: track 30.1 -> 23.1 mm
- net SCLK: track 11.7 -> 18.7 mm
- net 3V3: track 172.4 -> 165.6 mm, vias 8 -> 7
- net Net-(C2-Pad2): track 16.6 -> 10.0 mm
- net LCD_VDDI: track 11.7 -> 17.9 mm
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Other:
- board text added: "Author: Felix Neumann Date: 11/11/2025"
- board text added: "Board: Mini Arcade Mainboard V1.0"
- board text removed: "Board: Mini Arcade Mainboard V1.0 Author: Felix Neumann Date: 11/11/2025"

Commit message: 12 11 2025
Changed lines of the file:
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@@
 	)
 	(segment
-		(start 115.13 112.62)
-		(end 115.13 112.01295)
+		(start 114.52295 112.62)
+		(end 111.25 112.62)
 		(width 0.2)
 		(layer "F.Cu")
@@
 	)
 	(segment
-		(start 111.25 112.62)
-		(end 115.13 112.62)
-		(width 0.2)
-		(layer "F.Cu")
-		(net 19)
-	)
-	(segment
-		(start 115.13 112.01295)
+		(start 136.75 101.75)
 		(end 125.39295 101.75)
 		(width 0.2)
@@
 	)
 	(segment
-		(start 140.25 105.25)
-		(end 140.25 111.8375)
+		(start 125.39295 101.75)
+		(end 114.52295 112.62)
 		(width 0.2)
 		(layer "F.Cu")
@@
 	)
 	(segment
-		(start 136.75 101.75)
-		(end 140.25 105.25)
+		(start 140.25 105.25)
+		(end 136.75 101.75)
 		(width 0.2)
 		(layer "F.Cu")
@@
 	)
 	(segment
-		(start 125.39295 101.75)
-		(end 136.75 101.75)
+		(start 140.25 111.8375)
+		(end 140.25 105.25)
 		(width 0.2)
 		(layer "F.Cu")

Commit message: 14 11 2025
Other:
- board text added: "1"
- board text added: "5"
- board text added: "6"
Changed lines of the file:
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@@
 		(layer "Edge.Cuts")
+	)
+	(gr_text "1"
+		(at 113 115.75 0)
+		(layer "F.SilkS")
+		(effects
+			(font
+				(size 1 1)
+				(thickness 0.1)
+			)
+			(justify left bottom)
+		)
+	)
+	(gr_text "6\n"
+		(at 166 118.25 0)
+		(layer "F.SilkS")
+		(effects
+			(font
+				(size 1 1)
+				(thickness 0.1)
+			)
+			(justify left bottom)
+		)
 	)
 	(gr_text "Author: Felix Neumann\nDate:   11/11/2025\n"
@@
 			)
 			(justify left bottom)
+		)
+	)
+	(gr_text "1"
+		(at 166 105.5 0)
+		(layer "F.SilkS")
+		(effects
+			(font
+				(size 1 1)
+				(thickness 0.1)
+			)
+			(justify left bottom)
+		)
+	)
+	(gr_text "5"
+		(at 113 105.5 0)
+		(layer "F.SilkS")
+		(effects
+			(font
+				(size 1 1)
+				(thickness 0.1)
+			)
+			(justify left bottom)

Commit message: 17 11 2025
Connections:
- J2 pad 1: JS_UP -> GND
- J2 pad 2: JS_LEFT -> DP_UP
- J2 pad 3: JS_DOWN -> DP_RIGHT
- J2 pad 4: JS_SWITCH -> DP_DOWN
- J2 pad 5: JS_RIGHT -> DP_LEFT
- J3 pad 2: GND -> JS_UP
- J3 pad 3: DP_UP -> JS_LEFT
- J3 pad 4: DP_RIGHT -> JS_DOWN
- J3 pad 5: DP_DOWN -> JS_SWITCH
- J3 pad 6: DP_LEFT -> JS_RIGHT
- U1 pad 27: unconnected-(U1-PB14-Pad27) -> JS_RIGHT
- U1 pad 28: DP_LEFT -> JS_SWITCH
- U1 pad 29: DP_DOWN -> JS_DOWN
- U1 pad 30: DP_RIGHT -> JS_LEFT
- U1 pad 31: DP_UP -> JS_UP
- U1 pad 37: JS_RIGHT -> DP_LEFT
- U1 pad 38: JS_SWITCH -> DP_DOWN
- U1 pad 39: JS_DOWN -> DP_RIGHT
- U1 pad 40: JS_LEFT -> DP_UP
- U1 pad 41: JS_UP -> unconnected-(U1-PA20-Pad41)
Routing:
- net DP_LEFT: track 23.9 -> 48.2 mm
- net JS_RIGHT: track 48.2 -> 24.0 mm
- net DP_DOWN: track 23.1 -> 45.8 mm
- net JS_SWITCH: track 45.8 -> 23.3 mm
- net DP_RIGHT: track 24.0 -> 43.5 mm
- net JS_DOWN: track 43.5 -> 24.2 mm
- net DP_UP: track 24.8 -> 41.5 mm
- net JS_LEFT: track 41.5 -> 25.0 mm
- net JS_UP: track 38.6 -> 25.9 mm
- net GND: track 25.7 -> 25.9 mm, vias 25 -> 26
