File: MiniArcade_MainBoard/MiniArcade_MainBoard.kicad_pcb (KiCad board)
At the start: 2 copper layers, 60 x 55 mm, 31 parts, among them J1 62701021721, J2 Conn_01x05_Pin, J3 Conn_01x06_Pin, J4 F3311A7H121026E200, SW1 EVPAA, U1 ATSAMD21J18A-A, U2 LM321

Commit message: 19 11 2025
Changed lines of the file:
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@@
 	(footprint "Connector_PinHeader_2.54mm:PinHeader_1x06_P2.54mm_Vertical"
 		(layer "F.Cu")
-		(at 168.75 105)
+		(at 168.73 105)
 		(descr "Through hole straight pin header, 1x06, 2.54mm pitch, single row")
 		(tags "Through hole pin header THT 1x06 2.54mm single row")
@@
 	(footprint "Connector_PinHeader_2.54mm:PinHeader_1x05_P2.54mm_Vertical"
 		(layer "F.Cu")
-		(at 111.25 115.16 180)
+		(at 111.27 115.16 180)
 		(descr "Through hole straight pin header, 1x05, 2.54mm pitch, single row")
 		(tags "Through hole pin header THT 1x05 2.54mm single row")
@@
 		(hatch edge 0.5)
 		(connect_pads
-			(clearance 0.5)
+			(clearance 0.3)
 		)
 		(min_thickness 0.25)

Commit message: 26 11 2025
Routing:
- net GND: track 25.9 -> 33.2 mm, vias 26 -> 23
Other:
- board text added: "Author: Felix Neumann Date: Nov 2025"
- board text removed: "Author: Felix Neumann Date: 11/11/2025"
Changed lines of the file:
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@@
 		)
 	)
-	(gr_text "Author: Felix Neumann\nDate:   11/11/2025\n"
+	(gr_text "Author: Felix Neumann\nDate:   Nov 2025\n"
 		(at 142.75 101.75 0)
 		(layer "F.SilkS")
@@
 	)
 	(gr_text "Board: Mini Arcade Mainboard V1.0\n"
-		(at 120.5 95.25 0)
+		(at 120.25 93.5 0)
 		(layer "F.SilkS")
 		(effects
@@
 	)
 	(segment
+		(start 141.25 141.075)
+		(end 141.25 142.15)
+		(width 0.2)
+		(layer "F.Cu")
+		(net 2)
+	)
+	(segment
 		(start 137.299 141.776)
 		(end 138.201 141.776)
@@
 	)
 	(segment
+		(start 142.6 142.3)
+		(end 144.677 142.3)
+		(width 0.2)
+		(layer "F.Cu")
+		(net 2)
+	)
+	(segment
 		(start 162 141.45)
 		(end 161.201 140.651)
@@
 	)
 	(segment
+		(start 142.75 142.15)
+		(end 142.75 141.075)
+		(width 0.2)
+		(layer "F.Cu")
+		(net 2)
+	)
+	(segment
 		(start 143.75 118.75)
 		(end 145.6625 118.75)
@@
 	)
 	(segment
+		(start 145.25 141.727)
+		(end 145.25 141.075)
+		(width 0.2)
+		(layer "F.Cu")
+		(net 2)
+	)
+	(segment
 		(start 135.75 141.727)
 		(end 135.799 141.776)
@@
 	)
 	(segment
+		(start 141.25 142.15)
+		(end 141.4 142.3)
+		(width 0.2)
+		(layer "F.Cu")
+		(net 2)
+	)
+	(segment
 		(start 136.25 116.25)
 		(end 134.3375 116.25)
@@
 	)
 	(segment
+		(start 141.4 142.3)
+		(end 142.6 142.3)
+		(width 0.2)
+		(layer "F.Cu")
+		(net 2)
+	)
+	(segment
+		(start 144.677 142.3)
+		(end 145.25 141.727)
+		(width 0.2)
+		(layer "F.Cu")
+		(net 2)
+	)
+	(segment
 		(start 111.375 114.75)
 		(end 111.25 114.75)
@@
 	)
 	(segment
+		(start 142.6 142.3)
+		(end 142.75 142.15)
+		(width 0.2)
+		(layer "F.Cu")
+		(net 2)
+	)
+	(segment
 		(start 159 137.5375)
 		(end 158.9625 137.5)
@@
 	)
 	(via
-		(at 145.25 129.25)
-		(size 0.6)
-		(drill 0.3)
-		(layers "F.Cu" "B.Cu")
-		(free yes)
-		(net 2)
-	)
-	(via
 		(at 125 138.75)
 		(size 0.6)
@@
 	)
 	(via
-		(at 145.25 127.75)
-		(size 0.6)
-		(drill 0.3)
-		(layers "F.Cu" "B.Cu")
-		(free yes)
-		(net 2)
-	)
-	(via
 		(at 144.75 124.75)
 		(size 0.6)
@@
 	)
 	(via
-		(at 142.75 124.75)
+		(at 142.75 125.25)
 		(size 0.6)
 		(drill 0.3)
@@
 		(size 0.6)
 		(drill 0.3)
-		(layers "F.Cu" "B.Cu")
-		(free yes)
-		(net 2)
-	)
-	(via
-		(at 145.25 126.25)
-		(size 0.6)
-		(drill 0.3)
