File: MiniArcade_Controller/MiniArcade_Controller.kicad_pcb (KiCad board)
At the start: 2 copper layers, 55 x 25 mm, 7 parts, among them J1 Conn_01x05_Pin, J2 Conn_01x05_Pin, SW1 SW_Push_Dual_x2, SW2 SW_Push_Dual_x2, SW3 SW_Push_Dual_x2, SW4 SW_Push_Dual_x2

Commit message: 12 11 2025
Parts:
- J1, J2: footprint Connector_PinHeader_2.54mm:PinHeader_1x05_P2.54mm_Horizontal -> Connector_PinHeader_2.54mm:PinHeader_1x05_P2.54mm_Vertical
- moved J1 59.7 mm to (101.2, 109.9)
- moved S1 56.6 mm to (116.5, 115.0)
- moved SW3 52.1 mm to (139.2, 122.1)
- moved SW2 51.5 mm to (147.0, 112.8)
- moved SW4 51.5 mm to (131.5, 112.8)
- moved SW1 50.9 mm to (139.2, 103.4)
- moved J2 45.5 mm to (158.8, 109.9), turned to 180 degrees
Routing:
- net GND: track 0.00 -> 26.0 mm, vias 0 -> 4
- net DP_RIGHT: track 6.26 -> 11.9 mm
- net DP_UP: track 27.1 -> 22.2 mm
- net DP_DOWN: track 20.5 -> 24.9 mm, vias 0 -> 2
- net DP_LEFT: track 27.0 -> 31.1 mm
- net JS_DOWN: track 7.16 -> 10.8 mm, vias 1 -> 0
- net JS_LEFT: track 7.09 -> 10.7 mm, vias 1 -> 0
- net JS_UP: track 6.57 -> 10.1 mm, vias 1 -> 0
- net JS_RIGHT: track 20.0 -> 23.1 mm, vias 1 -> 2
- net JS_SWITCH: track 21.1 -> 23.6 mm, vias 1 -> 2
Other:
- board size 55 x 25 mm -> 60 x 30 mm

Commit message: 14 11 2025
Other:
- board text added: "1"
- board text added: "5"
Changed lines of the file:
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@@
 		(tags "Through hole pin header THT 1x05 2.54mm single row")
 		(property "Reference" "J2"
-			(at 0 2.67 -0)
+			(at 0 2.67 0)
 			(layer "F.SilkS")
 			(effects
@@
 		(tags "Through hole pin header THT 1x05 2.54mm single row")
 		(property "Reference" "J1"
-			(at 0 2.67 -0)
+			(at 0 2.67 0)
 			(layer "F.SilkS")
 			(effects
@@
 		(layer "Edge.Cuts")
 	)
+	(gr_text "1"
+		(at 156 110.5 0)
+		(layer "F.SilkS")
+		(effects
+			(font
+				(size 1 1)
+				(thickness 0.1)
+			)
+			(justify left bottom)
+		)
+	)
+	(gr_text "1"
+		(at 103.25 110.5 0)
+		(layer "F.SilkS")
+		(effects
+			(font
+				(size 1 1)
+				(thickness 0.1)
+			)
+			(justify left bottom)
+		)
+	)
+	(gr_text "5\n"
+		(at 103.25 120.75 0)
+		(layer "F.SilkS")
+		(effects
+			(font
+				(size 1 1)
+				(thickness 0.1)
+			)
+			(justify left bottom)
+		)
+	)
+	(gr_text "5\n"
+		(at 156 120.75 0)
+		(layer "F.SilkS")
+		(effects
+			(font
+				(size 1 1)
+				(thickness 0.1)
+			)
+			(justify left bottom)
+		)
+	)
 	(segment

Commit message: 19 11 2025
Changed lines of the file:
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@@
 	(footprint "Connector_PinHeader_2.54mm:PinHeader_1x05_P2.54mm_Vertical"
 		(layer "B.Cu")
-		(at 158.75 109.92 180)
+		(at 158.73 109.92 180)
 		(descr "Through hole straight pin header, 1x05, 2.54mm pitch, single row")
 		(tags "Through hole pin header THT 1x05 2.54mm single row")
@@
 	(footprint "Connector_PinHeader_2.54mm:PinHeader_1x05_P2.54mm_Vertical"
 		(layer "B.Cu")
-		(at 101.25 109.92 180)
+		(at 101.27 109.92 180)
 		(descr "Through hole straight pin header, 1x05, 2.54mm pitch, single row")
 		(tags "Through hole pin header THT 1x05 2.54mm single row")
@@
 	)
 	(segment
-		(start 156.54 119.75)
+		(start 156.46 117.54)
+		(end 154.25 119.75)
+		(width 0.2)
+		(layer "F.Cu")
+		(net 6)
+	)
+	(segment
+		(start 158.75 117.54)
+		(end 156.46 117.54)
+		(width 0.2)
+		(layer "F.Cu")
+		(net 6)
+	)
+	(segment
+		(start 154.25 119.75)
 		(end 145 119.75)
 		(width 0.2)
 		(layer "F.Cu")
-		(net 6)
-	)
-	(segment
-		(start 158.75 117.54)
-		(end 156.54 119.75)
-		(width 0.2)
-		(layer "F.Cu")

Commit message: 26 11 2025
Other:
- board text added: "Board: MiniArcade Controller Author: F.Neumann Date: Nov 2025"
Changed lines of the file:
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@@
+		)
+	)
+	(gr_text "Board:	MiniArcade Controller\nAuthor:	F.Neumann\nDate:	Nov 2025 \n"
+		(at 137.5 108.6 0)
+		(layer "B.SilkS")
+		(effects
+			(font
+				(size 1.5 1.5)
+				(thickness 0.3)
+				(bold yes)
+			)
+			(justify left bottom mirror)
 		)
 	)
