File: MiniArcade_PWR_Supply/MiniArcade_PWR_Supply/MiniArcade_PWR_Supply.kicad_pcb (KiCad board)
At the start: 2 copper layers, 53.5 x 55.2 mm, 17 parts, among them IC1 MIC94310-SYM5-TR, J1 Conn_01x03, J2 Conn_01x02_Pin, J3 Conn_01x02_Pin, U1 2479

Commit message: 05 11 2025
Changed lines of the file:
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@@
 			(effects
 				(font
-					(size 0.5 0.5)
-					(thickness 0.08)
+					(size 1 1)
+					(thickness 0.15)
 				)
 			)
@@
 			(effects
 				(font
-					(size 1.27 1.27)
-					(thickness 0.254)
+					(size 1 1)
+					(thickness 0.15)
 				)
 			)
@@
 			(effects
 				(font
-					(size 1.27 1.27)
-					(thickness 0.254)
+					(size 1 1)
+					(thickness 0.15)
 				)
 			)
@@
 			(effects
 				(font
-					(size 0.5 0.5)
-					(thickness 0.08)
+					(size 1 1)
+					(thickness 0.15)
 				)
 			)
@@
 			(effects
 				(font
-					(size 1.27 1.27)
-					(thickness 0.254)
+					(size 1 1)
+					(thickness 0.15)
 				)
 			)
@@
 			(effects
 				(font
-					(size 1.27 1.27)
-					(thickness 0.254)
+					(size 1 1)
+					(thickness 0.15)
 				)
 			)
@@
 			(effects
 				(font
-					(size 0.6 0.6)
-					(thickness 0.09)
+					(size 1 1)
+					(thickness 0.15)
 				)
 			)
@@
 			(effects
 				(font
-					(size 1.27 1.27)
-					(thickness 0.254)
+					(size 1 1)
+					(thickness 0.15)
 				)
 			)
@@
 			(effects
 				(font
-					(size 1.27 1.27)
-					(thickness 0.254)
+					(size 1 1)
+					(thickness 0.15)
 				)
 			)
@@
 			(effects
 				(font
-					(size 1.27 1.27)
-					(thickness 0.254)
+					(size 1 1)
+					(thickness 0.15)
 				)
 			)
@@
 			(effects
 				(font
-					(size 1.27 1.27)
-					(thickness 0.254)
+					(size 1 1)
+					(thickness 0.15)
 				)
 			)
@@
 			(effects
 				(font
-					(size 0.6 0.6)
-					(thickness 0.09)
+					(size 1 1)
+					(thickness 0.15)
 				)
 			)
@@
 			(effects
 				(font
-					(size 0.5 0.5)
-					(thickness 0.08)
+					(size 1 1)
+					(thickness 0.15)
 				)
 			)
@@
 			(effects
 				(font
-					(size 0.5 0.5)
-					(thickness 0.08)
+					(size 1 1)
+					(thickness 0.15)
 				)
 			)
@@
 			(effects
 				(font
-					(size 0.76 0.76)
-					(thickness 0.114)
+					(size 1 1)
+					(thickness 0.15)
 				)
 			)
@@
 			(effects
 				(font
-					(size 0.5 0.5)
-					(thickness 0.08)
+					(size 1 1)
+					(thickness 0.15)
 				)
 			)
@@
 			(effects
 				(font
-					(size 1.27 1.27)
-					(thickness 0.254)
+					(size 1 1)
+					(thickness 0.15)
 				)
 			)
@@
 			(effects
 				(font
-					(size 1.27 1.27)
-					(thickness 0.254)
+					(size 1 1)
+					(thickness 0.15)
 				)
 			)
@@
 			(effects
 				(font
-					(size 0.4 0.4)
-					(thickness 0.06)
+					(size 1 1)
+					(thickness 0.15)
 				)
 			)
@@
 			(effects
 				(font
-					(size 1.27 1.27)
-					(thickness 0.254)
+					(size 1 1)
+					(thickness 0.15)
 				)
 			)
@@
 			(effects
 				(font
-					(size 1.27 1.27)
-					(thickness 0.254)
+					(size 1 1)
+					(thickness 0.15)
 				)
 			)
@@
 			(effects
 				(font
-					(size 0.5 0.5)
-					(thickness 0.08)
+					(size 1 1)
+					(thickness 0.15)
 				)
 			)

Commit message: 10 11 2025
Parts:
- J2, J3: footprint Connector_PinHeader_1.00mm:PinHeader_1x02_P1.00mm_Horizontal -> Connector_PinHeader_2.54mm:PinHeader_1x02_P2.54mm_Horizontal
- moved J3 53.8 mm to (146.1, 49.3), turned to 180 degrees
- moved J2 18.9 mm to (191.8, 91.6)
- moved JP2 8.22 mm to (200.0, 86.5), turned to 90 degrees
- moved L1 7.90 mm to (198.8, 74.1), turned to -90 degrees
- moved C3 7.81 mm to (192.8, 85.5)
- moved IC1 7.81 mm to (192.8, 82.0)
- moved C1 4.52 mm to (188.7, 72.2)
- moved R4 4.37 mm to (196.8, 85.6), turned to 0 degrees
- moved R1 3.63 mm to (192.2, 65.8)
- moved C2 3.28 mm to (193.7, 74.5), turned to 180 degrees
- moved R2 3.06 mm to (192.2, 69.8)
- moved R3 3.06 mm to (192.2, 67.8)
- moved J1 1.96 mm to (190.7, 46.4)
- moved LED1 1.38 mm to (197.5, 82.8), turned to 180 degrees
- moved PS1 0.71 mm to (191.9, 72.3), turned to 0 degrees
Connections:
- J2 pad 1: GND -> 3V3
- J2 pad 2: 3V3 -> GND
Routing:
- net 5V0: track 2.23 -> 48.9 mm
- net Net-(PS1-EN): track 3.92 -> 22.6 mm
- net 3V5: track 16.8 -> 30.1 mm, vias 0 -> 2
- net GND: track 0.00 -> 6.56 mm, vias 0 -> 1
- net Net-(PS1-FB): track 6.28 -> 12.0 mm
- net 3V3: track 7.03 -> 11.6 mm
- net 4V5: track 9.27 -> 11.3 mm
- net Net-(PS1-SW): track 4.49 -> 6.29 mm
- net Net-(JP2-B): track 2.35 -> 3.57 mm
- added copper zone on F.Cu, net 3V5
- added copper zone on B.Cu, net GND
- added copper zone on F.Cu, net GND
- added copper zone on F.Cu, net Net-(PS1-EN)
- added copper zone on F.Cu, net Net-(PS1-FB)
- added copper zone on F.Cu, net Net-(PS1-SW)
Other:
- board size 53.5 x 55.2 mm -> 66.4 x 55.2 mm
- board text added: "Board: MiniArcade Powersupply V1.0 Author: Felix Neumann Date: 11/08/2025"

Commit message: 11 11 2025
Parts:
- J2, J3: footprint Connector_PinHeader_2.54mm:PinHeader_1x02_P2.54mm_Horizontal -> Connector_PinHeader_2.54mm:PinHeader_1x02_P2.54mm_Vertical
- moved J2 9.07 mm to (200.7, 93.4)
- moved J3 3.08 mm to (143.3, 48.1)
Routing:
- net 3V3: track 11.6 -> 17.7 mm
- net 5V0: track 48.9 -> 51.0 mm
Other:
- board size 66.4 x 55.2 mm -> 60 x 55.2 mm
- board text added: "Board: MiniArcade Powersupply V1.0 Author: F.Neumann Date: 11/08/2025"
- board text removed: "Board: MiniArcade Powersupply V1.0 Author: Felix Neumann Date: 11/08/2025"

Commit message: 14 11 2025
Parts:
- moved J2 102.9 mm to (101.2, 120.0)
- moved J3 76.0 mm to (158.8, 122.5)
- moved C1 71.4 mm to (146.7, 130.0)
- moved C2 71.4 mm to (151.7, 132.3)
- moved C3 71.4 mm to (150.8, 143.3)
- moved IC1 71.4 mm to (150.8, 139.8)
- moved J1 71.4 mm to (148.7, 104.2)
- moved JP2 71.4 mm to (158.0, 144.2)
- moved L1 71.4 mm to (156.8, 131.9)
- moved LED1 71.4 mm to (155.5, 140.6)
- moved PS1 71.4 mm to (149.9, 130.1)
- moved R1 71.4 mm to (150.2, 123.6)
- moved R2 71.4 mm to (150.2, 127.6)
- moved R3 71.4 mm to (150.2, 125.6)
- moved R4 71.4 mm to (154.8, 143.3)
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Routing:
- net 3V3: track 17.7 -> 66.3 mm
- net 5V0: track 51.0 -> 21.6 mm
Other:
- board size 60 x 55.2 mm -> 60 x 55 mm
- board text added: "1"
- board text added: "2"
- board text added: "Board: MiniArcade PWR-SPLY V1.0 Author: F.Neumann Date: Nov. 2025"
- board text removed: "Board: MiniArcade Powersupply V1.0 Author: F.Neumann Date: 11/08/2025"

Commit message: 17 11 2025
Connections:
- J2 pad 1: 3V3 -> GND
- J2 pad 2: GND -> 5V0
- J3 pad 1: GND -> 3V3
- J3 pad 2: 5V0 -> GND
Routing:
- net 5V0: track 21.6 -> 59.6 mm
- net 3V3: track 66.3 -> 33.8 mm, vias 0 -> 2
Changed lines of the file:
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@@
 			(layers "*.Cu" "*.Mask")
 			(remove_unused_layers no)
-			(net 4 "3V3")
+			(net 1 "GND")
 			(pinfunction "Pin_1")
 			(pintype "passive")
@@
 			(layers "*.Cu" "*.Mask")
 			(remove_unused_layers no)
-			(net 1 "GND")
+			(net 7 "5V0")
 			(pinfunction "Pin_2")
 			(pintype "passive")
@@
 			(layers "*.Cu" "*.Mask")
 			(remove_unused_layers no)
-			(net 1 "GND")
+			(net 4 "3V3")
 			(pinfunction "Pin_1")
 			(pintype "passive")
@@
 			(layers "*.Cu" "*.Mask")
 			(remove_unused_layers no)
-			(net 7 "5V0")
+			(net 1 "GND")
 			(pinfunction "Pin_2")
 			(pintype "passive")
@@
 		(tags "Through hole pin header THT 1x03 1.00mm single row")
 		(property "Reference" "J1"
-			(at 1.9 1.3 180)
+			(at 0.15 4.05 180)
 			(layer "F.SilkS")
 			(effects
@@
 	)
 	(gr_text "2"
-		(at 155.5 123.25 0)
+		(at 155.75 120.5 0)
 		(layer "F.SilkS")
 		(effects
@@
 	)
 	(gr_text "1\n"
-		(at 155.5 120.5 0)
+		(at 155.75 123.25 0)
+		(layer "F.SilkS")
+		(effects
+			(font
+				(size 1 1)
+				(thickness 0.1)
+			)
+			(justify left bottom)
+		)
+	)
+	(gr_text "1\n"
+		(at 103.75 120.5 0)
+		(layer "F.SilkS")
+		(effects
+			(font
+				(size 1 1)
+				(thickness 0.1)
+			)
+			(justify left bottom)
+		)
+	)
+	(gr_text "2"
+		(at 103.75 123.25 0)
 		(layer "F.SilkS")
 		(effects
@@
 	)
 	(segment
-		(start 150.0875 145)
-		(end 126.25 145)
+		(start 151.7 142.25)
+		(end 151.7 141.05)
 		(width 0.2)
 		(layer "F.Cu")
@@
 	)
 	(segment
-		(start 151.7 142.25)
-		(end 151.7 141.05)
+		(start 158.75 122.54)
+		(end 158.75 126.5)
 		(width 0.2)
 		(layer "F.Cu")
@@
 	(segment
 		(start 151.7875 143.3)
-		(end 150.0875 145)
+		(end 151.45 143.3)
 		(width 0.2)
 		(layer "F.Cu")
@@
 	)
 	(segment
-		(start 151.7875 143.3)
-		(end 151.45 143.3)
+		(start 151.7875 145.9625)
+		(end 151.7875 143.3)
 		(width 0.2)
 		(layer "F.Cu")
@@
 	)
 	(segment
-		(start 126.25 145)
-		(end 101.25 120)
+		(start 151.75 146)
+		(end 151.7875 145.9625)
 		(width 0.2)
 		(layer "F.Cu")
@@
 		(net 4)
 	)
+	(via
+		(at 158.75 126.5)
+		(size 0.6)
+		(drill 0.3)
+		(layers "F.Cu" "B.Cu")
+		(net 4)
+	)
+	(via
+		(at 151.75 146)
+		(size 0.6)
+		(drill 0.3)
+		(layers "F.Cu" "B.Cu")
+		(net 4)
+	)
+	(segment
+		(start 158.75 126.5)
+		(end 158.75 139)
+		(width 0.2)
+		(layer "B.Cu")
+		(net 4)
+	)
+	(segment
+		(start 158.75 139)
+		(end 151.75 146)
+		(width 0.2)
+		(layer "B.Cu")
+		(net 4)
+	)
 	(segment
 		(start 148.75 103.97328)
@@
 	)
 	(segment
-		(start 156.75 106)
-		(end 154.9 104.15)
+		(start 148.65104 101.5)
+		(end 150.7 103.54896)
 		(width 0.2)
 		(layer "F.Cu")
@@
 	)
 	(segment
-		(start 154.9 104.15)
-		(end 150.7 104.15)
+		(start 122.29 101.5)
+		(end 148.65104 101.5)
 		(width 0.2)
 		(layer "F.Cu")
@@
 	)
 	(segment
-		(start 156.75 118)
-		(end 156.75 106)
+		(start 101.25 122.54)
+		(end 122.29 101.5)
 		(width 0.2)
 		(layer "F.Cu")
@@
 	)
 	(segment
-		(start 158.75 120)
-		(end 156.75 118)
+		(start 150.7 103.54896)
+		(end 150.7 104.15)
 		(width 0.2)
 		(layer "F.Cu")

Commit message: 19 11 2025
Routing:
- net 3V5: track 30.1 -> 35.7 mm, vias 2 -> 4
- net GND: track 6.56 -> 10.2 mm
- net Net-(PS1-EN): track 22.6 -> 25.9 mm, vias 0 -> 2
- net Net-(PS1-FB): track 12.0 -> 13.4 mm

Commit message: 08 12 2025
Routing:
- net Net-(PS1-FB): track 13.4 -> 6.05 mm
Changed lines of the file:
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@@
+	)
+	(segment
+		(start 149.167926 127.582074)
+		(end 149.167926 129.381074)
+		(width 0.7)
+		(layer "F.Cu")
+		(net 12)
 	)
 	(segment
@@
 	)
 	(segment
-		(start 149.167926 125.582074)
-		(end 149.167926 123.582074)
-		(width 0.2)
+		(start 149.1 127.514148)
+		(end 149.1 125.65)
+		(width 1)
 		(layer "F.Cu")
 		(net 12)
 	)
 	(segment
-		(start 148.301 129.351)
-		(end 148.301 127.95)
-		(width 0.2)
-		(layer "F.Cu")
-		(net 12)
-	)
-	(segment
-		(start 148.8 127.95)
-		(end 149.167926 127.582074)
-		(width 0.2)
-		(layer "F.Cu")
-		(net 12)
-	)
-	(segment
-		(start 148.532074 129.582074)
-		(end 148.301 129.351)
-		(width 0.2)
-		(layer "F.Cu")
-		(net 12)
-	)
-	(segment
-		(start 148.301 127.95)
-		(end 148.8 127.95)
-		(width 0.2)
-		(layer "F.Cu")
-		(net 12)
-	)
-	(segment
-		(start 149.117926 129.582074)
-		(end 149.117926 123.632074)
+		(start 149.167926 129.532074)
+		(end 149.117926 129.582074)
 		(width 0.2)
 		(layer "F.Cu")
@@
 	(segment
 		(start 149.167926 127.582074)
-		(end 149.167926 125.582074)
-		(width 0.2)
+		(end 149.1 127.514148)
+		(width 1)
 		(layer "F.Cu")
 		(net 12)
 	)
 	(segment
-		(start 149.117926 129.582074)
-		(end 148.532074 129.582074)
-		(width 0.2)
+		(start 149.167926 125.582074)
+		(end 149.167926 123.582074)
+		(width 1)
+		(layer "F.Cu")
+		(net 12)
+	)
+	(segment
+		(start 149.167926 129.381074)
+		(end 149.117926 129.381074)
+		(width 0.7)
+		(layer "F.Cu")
+		(net 12)
+	)
+	(segment
+		(start 149.1 125.65)
+		(end 149.167926 125.582074)
+		(width 1)
 		(layer "F.Cu")
 		(net 12)
@@
 			(thermal_gap 0.5)
 			(thermal_bridge_width 0.5)
-			(island_removal_mode 1)
-			(island_area_min 9.999999)
 		)
 		(polygon
