File: MiniArcade_Left_Sidepanel/MiniArcade_Left_Sidepanel.kicad_pcb (KiCad board)
At the start: 2 copper layers, 50 x 100 mm, 6 parts, among them J1 M20-7910242R, J2 M20-7910542R, J3 M20-7910642R, J4 USB_C_PWR_Connector

Commit message: 19 11 2025
Parts:
- removed J4: USB_C_PWR_Connector, MiniArcadeLeftSidepanel:USB4125GFA
- removed R5, R6: 5k1, Resistor_SMD:R_0603_1608Metric_Pad0.98x0.95mm_HandSolder
- J1, J2, J3: moved to B.Cu
- moved J3 71.9 mm to (91.6, 96.3), turned to 90 degrees
- moved J1 1.33 mm to (133.2, 141.2), turned to -90 degrees
- moved J2 0.92 mm to (125.0, 128.8), turned to 180 degrees
Connections:
- J1 pad 1: GND -> 3V3
- J1 pad 2: 5V0 -> GND
- J2 pad 1: GND -> JS_RIGHT
- J2 pad 2: DP_UP -> JS_SWITCH
- J2 pad 3: DP_RIGHT -> JS_DOWN
- J2 pad 4: DP_DOWN -> JS_LEFT
- J2 pad 5: DP_LEFT -> JS_UP
- J3 pad 1: 3V3 -> JS_RIGHT
- J3 pad 2: JS_UP -> JS_SWITCH
- J3 pad 3: JS_LEFT -> JS_DOWN
- J3 pad 4: JS_DOWN -> JS_LEFT
- J3 pad 5: JS_SWITCH -> JS_UP
- J3 pad 6: JS_RIGHT -> 3V3
Routing:
- net 3V3: track 0.00 -> 102.0 mm
- net JS_LEFT: track 0.00 -> 85.0 mm, vias 0 -> 2
- net JS_DOWN: track 0.00 -> 84.8 mm, vias 0 -> 2
- net JS_SWITCH: track 0.00 -> 84.7 mm, vias 0 -> 2
- net JS_UP: track 0.00 -> 84.4 mm
- net JS_RIGHT: track 0.00 -> 80.9 mm, vias 0 -> 2
- added copper zone on B.Cu, net GND
- added copper zone on F.Cu, net GND
Other:
- board size 50 x 100 mm -> 60 x 100 mm
- board text added: "1"
- board text added: "2"
- board text added: "5"
- board text added: "6"
- board text added: "Board: MiniArcade Right Side Panel Author: Felix Neumann Date: Nov. 2025"

Commit message: 21 11 2025
Parts:
- added ?: , , F.Cu at (123.6, 79.0)
Other:
- outline, holes or cut-outs redrawn
Changed lines of the file:
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@@
 	(net 6 "JS_SWITCH")
 	(net 7 "3V3")
+	(footprint ""
+		(layer "F.Cu")
+		(at 123.6 79 90)
+		(property "Reference" ""
+			(at 0 0 90)
+			(layer "F.SilkS")
+			(effects
+				(font
+					(size 1.27 1.27)
+					(thickness 0.15)
+				)
+			)
+		)
+		(property "Value" ""
+			(at 0 0 90)
+			(layer "F.Fab")
+			(effects
+				(font
+					(size 1.27 1.27)
+					(thickness 0.15)
+				)
+			)
+		)
+		(property "Datasheet" ""
+			(at 0 0 90)
+			(layer "F.Fab")
+			(hide yes)
+			(effects
+				(font
+					(size 1.27 1.27)
+					(thickness 0.15)
+				)
+			)
+		)
+		(property "Description" ""
+			(at 0 0 90)
+			(layer "F.Fab")
+			(hide yes)
+			(effects
+				(font
+					(size 1.27 1.27)
+					(thickness 0.15)
+				)
+			)
+		)
+		(pad "" smd rect
+			(at 0 -0.1 180)
+			(size 3 8)
+			(layers "B.Cu" "B.Mask" "B.Paste")
+			(pinfunction "6")
+			(pintype "passive")
+		)
+		(embedded_fonts no)
+	)
 	(footprint "MiniArcadeLeftSidepanel:M207910542R"
 		(layer "B.Cu")
@@
 	)
 	(gr_line
+		(start 125 80.25)
+		(end 126.6 80.25)
+		(stroke
+			(width 0.05)
+			(type solid)
+		)
+		(layer "Edge.Cuts")
+	)
+	(gr_line
 		(start 110 120)
 		(end 110 100)
@@
 	)
 	(gr_line
-		(start 125 75)
-		(end 125 80)
-		(stroke
-			(width 0.05)
-			(type solid)
+		(start 110 100)
+		(end 125 83)
+		(stroke
+			(width 0.05)
+			(type default)
 		)
 		(layer "Edge.Cuts")
@@
 	)
 	(gr_line
+		(start 125 83)
+		(end 125 80.25)
+		(stroke
+			(width 0.05)
+			(type default)
+		)
+		(layer "Edge.Cuts")
+	)
+	(gr_line
 		(start 80 175)
 		(end 80 80)
@@
 	)
 	(gr_line
-		(start 110 100)
-		(end 125 80)
-		(stroke
-			(width 0.05)
-			(type default)
+		(start 126.6 80.25)
+		(end 126.6 77.75)
+		(stroke
+			(width 0.05)
+			(type solid)
 		)
 		(layer "Edge.Cuts")
@@
 		(stroke
 			(width 0.05)
+			(type default)
+		)
+		(layer "Edge.Cuts")
+	)
+	(gr_line
+		(start 125 77.75)
+		(end 126.6 77.75)
+		(stroke
+			(width 0.05)
+			(type solid)
+		)
+		(layer "Edge.Cuts")
+	)
+	(gr_line
+		(start 125 77.75)
+		(end 125 75)
+		(stroke
+			(width 0.05)

Commit message: 25 11 2025
Parts:
- added ?: , , F.Cu at (89.0, 76.5)
Other:
- board size 60 x 100 mm -> 60 x 101.5 mm
Changed lines of the file:
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@@
+	(footprint ""
+		(layer "F.Cu")
+		(at 89 76.5 90)
+		(property "Reference" ""
+			(at 0 0 90)
+			(layer "F.SilkS")
+			(effects
+				(font
+					(size 1.27 1.27)
+					(thickness 0.15)
+				)
+			)
+		)
+		(property "Value" ""
+			(at 0 0 90)
+			(layer "F.Fab")
+			(effects
+				(font
+					(size 1.27 1.27)
+					(thickness 0.15)
+				)
+			)
+		)
+		(property "Datasheet" ""
+			(at 0 0 90)
+			(layer "F.Fab")
+			(hide yes)
+			(effects
+				(font
+					(size 1.27 1.27)
+					(thickness 0.15)
+				)
+			)
+		)
+		(property "Description" ""
+			(at 0 0 90)
+			(layer "F.Fab")
+			(hide yes)
+			(effects
+				(font
+					(size 1.27 1.27)
+					(thickness 0.15)
+				)
+			)
+		)
+		(pad "" smd rect
+			(at 0 0 270)
+			(size 3 8)
+			(layers "B.Cu" "B.Mask" "B.Paste")
+			(pinfunction "6")
+			(pintype "passive")
+		)
+		(embedded_fonts no)
+	)
 	(footprint ""
 		(layer "F.Cu")
@@
 	)
 	(gr_line
+		(start 95.5 73.5)
+		(end 95.5 75)
+		(stroke
+			(width 0.05)
+			(type default)
+		)
+		(layer "Edge.Cuts")
+	)
+	(gr_line
 		(start 125 80.25)
 		(end 126.6 80.25)
@@
 	)
 	(gr_line
+		(start 90.5 73.5)
+		(end 95.5 73.5)
+		(stroke
+			(width 0.05)
+			(type default)
+		)
+		(layer "Edge.Cuts")
+	)
+	(gr_line
 		(start 140 175)
 		(end 80 175)
@@
 	)
 	(gr_line
-		(start 125 75)
-		(end 85 75)
+		(start 95.5 75)
+		(end 125 75)
 		(stroke
 			(width 0.05)
-			(type solid)
+			(type default)
+		)
+		(layer "Edge.Cuts")
+	)
+	(gr_line
+		(start 85 75)
+		(end 90.5 75)
+		(stroke
+			(width 0.05)
+			(type default)
 		)
 		(layer "Edge.Cuts")
@@
 			(width 0.05)
 			(type solid)
+		)
+		(layer "Edge.Cuts")
+	)
+	(gr_line
+		(start 90.5 75)
+		(end 90.5 73.5)
+		(stroke
+			(width 0.05)
+			(type default)
 		)
 		(layer "Edge.Cuts")
@@
 		(polygon
 			(pts
-				(xy 80 75) (xy 80 175) (xy 140 175) (xy 140 75)
-			)
-		)
+				(xy 80 72.5) (xy 80 175) (xy 140 175) (xy 140 72.5)
+			)
+		)
