File: MiniArcade_Top_Cover/MiniArcade_Top_Cover.kicad_pcb (KiCad board)
At the start: 2 copper layers, 63 x 41.5 mm, 0 parts

Commit message: 25 11 2025
Parts:
- added ?: , , B.Cu at (169.8, 55.5)
- added ?: , , B.Cu at (113.2, 55.5)
Changed lines of the file:
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@@
 	)
 	(net 0 "")
+	(footprint ""
+		(layer "B.Cu")
+		(at 169.8 55.5 180)
+		(property "Reference" ""
+			(at 0 0 0)
+			(layer "B.SilkS")
+			(effects
+				(font
+					(size 1.27 1.27)
+					(thickness 0.15)
+				)
+				(justify mirror)
+			)
+		)
+		(property "Value" ""
+			(at 0 0 0)
+			(layer "B.Fab")
+			(effects
+				(font
+					(size 1.27 1.27)
+					(thickness 0.15)
+				)
+				(justify mirror)
+			)
+		)
+		(property "Datasheet" ""
+			(at 0 0 0)
+			(layer "B.Fab")
+			(hide yes)
+			(effects
+				(font
+					(size 1.27 1.27)
+					(thickness 0.15)
+				)
+				(justify mirror)
+			)
+		)
+		(property "Description" ""
+			(at 0 0 0)
+			(layer "B.Fab")
+			(hide yes)
+			(effects
+				(font
+					(size 1.27 1.27)
+					(thickness 0.15)
+				)
+				(justify mirror)
+			)
+		)
+		(pad "" smd rect
+			(at 0 0)
+			(size 3 8)
+			(layers "F.Cu" "F.Mask" "F.Paste")
+			(pinfunction "6")
+			(pintype "passive")
+		)
+		(embedded_fonts no)
+	)
+	(footprint ""
+		(layer "B.Cu")
+		(at 113.2 55.5 180)
+		(property "Reference" ""
+			(at 0 0 0)
+			(layer "B.SilkS")
+			(effects
+				(font
+					(size 1.27 1.27)
+					(thickness 0.15)
+				)
+				(justify mirror)
+			)
+		)
+		(property "Value" ""
+			(at 0 0 0)
+			(layer "B.Fab")
+			(effects
+				(font
+					(size 1.27 1.27)
+					(thickness 0.15)
+				)
+				(justify mirror)
+			)
+		)
+		(property "Datasheet" ""
+			(at 0 0 0)
+			(layer "B.Fab")
+			(hide yes)
+			(effects
+				(font
+					(size 1.27 1.27)
+					(thickness 0.15)
+				)
+				(justify mirror)
+			)
+		)
+		(property "Description" ""
+			(at 0 0 0)
+			(layer "B.Fab")
+			(hide yes)
+			(effects
+				(font
+					(size 1.27 1.27)
+					(thickness 0.15)
+				)
+				(justify mirror)
+			)
+		)
+		(pad "" smd rect
+			(at 0 0)
+			(size 3 8)
+			(layers "F.Cu" "F.Mask" "F.Paste")
+			(pinfunction "6")
+			(pintype "passive")
+		)
+		(embedded_fonts no)
+	)
 	(gr_line
 		(start 173 51.5)
