File: MiniArcade_Right_Sidepanel/MiniArcade_Right_Sidepanel.kicad_pcb (KiCad board)
At the start: 2 copper layers, 60 x 100 mm, 6 parts, among them J1 M20-7910242R, J2 M20-7910542R, J3 M20-7910542R

Commit message: 21 11 2025
Parts:
- added ?: , , B.Cu at (123.5, 79.0)
Other:
- outline, holes or cut-outs redrawn
Changed lines of the file:
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@@
 		)
+	)
+	(footprint ""
+		(layer "B.Cu")
+		(at 123.5 79 180)
+		(property "Reference" ""
+			(at 0 0 0)
+			(layer "B.SilkS")
+			(effects
+				(font
+					(size 1.27 1.27)
+					(thickness 0.15)
+				)
+				(justify mirror)
+			)
+		)
+		(property "Value" ""
+			(at 0 0 0)
+			(layer "B.Fab")
+			(effects
+				(font
+					(size 1.27 1.27)
+					(thickness 0.15)
+				)
+				(justify mirror)
+			)
+		)
+		(property "Datasheet" ""
+			(at 0 0 0)
+			(layer "B.Fab")
+			(hide yes)
+			(effects
+				(font
+					(size 1.27 1.27)
+					(thickness 0.15)
+				)
+				(justify mirror)
+			)
+		)
+		(property "Description" ""
+			(at 0 0 0)
+			(layer "B.Fab")
+			(hide yes)
+			(effects
+				(font
+					(size 1.27 1.27)
+					(thickness 0.15)
+				)
+				(justify mirror)
+			)
+		)
+		(pad "" smd rect
+			(at 0 0 270)
+			(size 8 3)
+			(layers "F.Cu" "F.Mask" "F.Paste")
+			(pinfunction "6")
+			(pintype "passive")
+		)
+		(embedded_fonts no)
+	)
+	(gr_line
+		(start 126.6 80.25)
+		(end 126.6 77.75)
+		(stroke
+			(width 0.05)
+			(type default)
+		)
+		(layer "Edge.Cuts")
 	)
 	(gr_line
@@
 	(gr_line
 		(start 125 75)
-		(end 125 80)
+		(end 125 77.75)
 		(stroke
 			(width 0.05)
-			(type solid)
+			(type default)
 		)
 		(layer "Edge.Cuts")
@@
 	)
 	(gr_line
+		(start 125 83)
+		(end 125 80.25)
+		(stroke
+			(width 0.05)
+			(type default)
+		)
+		(layer "Edge.Cuts")
+	)
+	(gr_line
 		(start 140 175)
 		(end 80 175)
@@
 	)
 	(gr_line
-		(start 110 100)
-		(end 125 80)
+		(start 125 80.25)
+		(end 126.6 80.25)
 		(stroke
 			(width 0.05)
-			(type default)
+			(type solid)
+		)
+		(layer "Edge.Cuts")
+	)
+	(gr_line
+		(start 125 77.75)
+		(end 126.6 77.75)
+		(stroke
+			(width 0.05)
+			(type solid)
 		)
 		(layer "Edge.Cuts")
@@
 		)
 		(layer "Edge.Cuts")
+	)
+	(gr_line
+		(start 110 100)
+		(end 125 83)
+		(stroke
+			(width 0.05)
+			(type default)
+		)
+		(layer "Edge.Cuts")

Commit message: 25 11 2025
Parts:
- added ?: , , F.Cu at (89.0, 76.5)
Other:
- board size 60 x 100 mm -> 60 x 101.5 mm
Changed lines of the file:
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@@
+	)
+	(footprint ""
+		(layer "F.Cu")
+		(at 89 76.5 90)
+		(property "Reference" ""
+			(at 0 0 90)
+			(layer "F.SilkS")
+			(effects
+				(font
+					(size 1.27 1.27)
+					(thickness 0.15)
+				)
+			)
+		)
+		(property "Value" ""
+			(at 0 0 90)
+			(layer "F.Fab")
+			(effects
+				(font
+					(size 1.27 1.27)
+					(thickness 0.15)
+				)
+			)
+		)
+		(property "Datasheet" ""
+			(at 0 0 90)
+			(layer "F.Fab")
+			(hide yes)
+			(effects
+				(font
+					(size 1.27 1.27)
+					(thickness 0.15)
+				)
+			)
+		)
+		(property "Description" ""
+			(at 0 0 90)
+			(layer "F.Fab")
+			(hide yes)
+			(effects
+				(font
+					(size 1.27 1.27)
+					(thickness 0.15)
+				)
+			)
+		)
+		(pad "" smd rect
+			(at 0 0)
+			(size 8 3)
+			(layers "F.Cu" "F.Mask" "F.Paste")
+			(pinfunction "6")
+			(pintype "passive")
+		)
+		(embedded_fonts no)
 	)
 	(footprint ""
@@
 	)
 	(gr_line
-		(start 125 75)
-		(end 85 75)
-		(stroke
-			(width 0.05)
-			(type solid)
+		(start 85 75)
+		(end 90.5 75)
+		(stroke
+			(width 0.05)
+			(type default)
+		)
+		(layer "Edge.Cuts")
+	)
+	(gr_line
+		(start 95.5 75)
+		(end 125 75)
+		(stroke
+			(width 0.05)
+			(type default)
 		)
 		(layer "Edge.Cuts")
@@
 	)
 	(gr_line
+		(start 90.5 75)
+		(end 90.5 73.5)
+		(stroke
+			(width 0.05)
+			(type default)
+		)
+		(layer "Edge.Cuts")
+	)
+	(gr_line
 		(start 125 80.25)
 		(end 126.6 80.25)
@@
 	)
 	(gr_line
+		(start 90.5 73.5)
+		(end 95.5 73.5)
+		(stroke
+			(width 0.05)
+			(type default)
+		)
+		(layer "Edge.Cuts")
+	)
+	(gr_line
 		(start 110 120)
 		(end 110 100)
@@
 		)
 		(layer "Edge.Cuts")
+	)
+	(gr_line
+		(start 95.5 73.5)
+		(end 95.5 75)
+		(stroke
+			(width 0.05)
+			(type default)
+		)
+		(layer "Edge.Cuts")

Commit message: 26 11 2025
Routing:
- net 5V0: track 40.4 -> 45.0 mm
Changed lines of the file:
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@@
 			(effects
 				(font
-					(size 1.27 1.27)
-					(thickness 0.254)
+					(size 1 1)
+					(thickness 0.15)
 				)
 			)
@@
 			(effects
 				(font
-					(size 1.27 1.27)
-					(thickness 0.254)
+					(size 1 1)
+					(thickness 0.15)
 				)
 			)
@@
 			(effects
 				(font
-					(size 1.27 1.27)
-					(thickness 0.254)
+					(size 1 1)
+					(thickness 0.15)
 				)
 			)
@@
 			(effects
 				(font
-					(size 1.27 1.27)
-					(thickness 0.254)
+					(size 1 1)
+					(thickness 0.15)
 				)
 			)
@@
 			(effects
 				(font
-					(size 1.27 1.27)
-					(thickness 0.254)
+					(size 1 1)
+					(thickness 0.15)
 				)
 			)
@@
 			(effects
 				(font
-					(size 1.27 1.27)
-					(thickness 0.254)
+					(size 1 1)
+					(thickness 0.15)
 				)
 			)
@@
 			(effects
 				(font
-					(size 1.27 1.27)
+					(size 1 1)
 					(thickness 0.15)
 				)
@@
 	)
 	(gr_text "Board:	MiniArcade Right Side Panel\nAuthor:	Felix Neumann\nDate:	Nov. 2025\n"
-		(at 82.5 172.25 -0)
+		(at 82.5 172.25 0)
 		(layer "F.SilkS")
 		(effects
@@
 		(effects
 			(font
-				(size 1.5 1.5)
-				(thickness 0.3)
+				(size 1 1)
+				(thickness 0.15)
 				(bold yes)
 			)
@@
 		(effects
 			(font
-				(size 1.5 1.5)
-				(thickness 0.3)
+				(size 1 1)
+				(thickness 0.15)
 				(bold yes)
 			)
@@
 		(effects
 			(font
-				(size 1.5 1.5)
-				(thickness 0.3)
+				(size 1 1)
+				(thickness 0.15)
 				(bold yes)
 			)
@@
 		(effects
 			(font
-				(size 1.5 1.5)
-				(thickness 0.3)
+				(size 1 1)
+				(thickness 0.15)
 				(bold yes)
 			)
@@
 		(effects
 			(font
-				(size 1.5 1.5)
-				(thickness 0.3)
+				(size 1 1)
+				(thickness 0.15)
 				(bold yes)
 			)
@@
 		(effects
 			(font
-				(size 1.5 1.5)
-				(thickness 0.3)
+				(size 1 1)
+				(thickness 0.15)
 				(bold yes)
 			)
@@
 	)
 	(segment
+		(start 85.996 142.23)
+		(end 85.5 142.726)
+		(width 0.2)
+		(layer "F.Cu")
+		(net 4)
+	)
+	(segment
+		(start 85.5 142.726)
+		(end 85.5 145)
+		(width 0.2)
+		(layer "F.Cu")
+		(net 4)
+	)
+	(segment
+		(start 85.77 145.27)
+		(end 86.528 145.27)
+		(width 0.2)
+		(layer "F.Cu")
+		(net 4)
+	)
+	(segment
+		(start 85.5 145)
+		(end 85.77 145.27)
+		(width 0.2)
+		(layer "F.Cu")
+		(net 4)
+	)
+	(segment
 		(start 88.02 142.23)
 		(end 89.25 141)
 		(width 0.2)
 		(layer "F.Cu")
+		(net 4)
+	)
+	(segment
+		(start 86.528 142.23)
+		(end 85.996 142.23)
+		(width 0.2)
+		(layer "F.Cu")
